Commit message: refactor: Add RTAB-Map Package
Add RTAB-Map Package
Upgrade sensor
Add mapping.launch
Remove videos

File: catkin_ws/src/my_robot/urdf/my_robot.xacro (robot description, xacro)
@@ -184,3 +184,10 @@
     <dynamics damping="1.0" friction="1.0"/>
   </joint>
+  <joint name="camera_optical_joint" type="fixed">
+    <origin xyz="0 0 0" rpy="-1.5707 0 -1.5707"/>
+    <parent link="camera"/>
+    <child link="camera_link_optical"/>
+  </joint>
+  <link name="camera_link_optical">
+  </link>
 </robot>
